File: Proyecto-diseño-PCB/Proyecto-diseño-PCB.kicad_sch (KiCad schematic)
At the start: 41 parts, among them J1 Conn_01x13_Pin, J2 PROGRAMACIÓN/DEPURACIÓN, J3 USB_B_Micro, J4 Conn_01x13_Pin, SW1 RESET, SW2 BOTON, SW3 BOTON, U1 PIC18LF45K50-I/P, U2 LP2950-3.3_TO92, U3 TPD2EUSB30

Commit message: Asignación de footprints
Parts:
- C1: renamed from C7; footprint (none) -> Capacitor_THT:C_Disc_D3.4mm_W2.1mm_P2.50mm
- C2: renamed from C8; footprint (none) -> Capacitor_THT:C_Disc_D3.4mm_W2.1mm_P2.50mm
- C3: renamed from C1; footprint (none) -> Capacitor_THT:C_Disc_D3.4mm_W2.1mm_P2.50mm
- C4: footprint (none) -> Capacitor_THT:C_Disc_D3.4mm_W2.1mm_P2.50mm
- C5: renamed from C6; footprint (none) -> Capacitor_THT:C_Disc_D3.4mm_W2.1mm_P2.50mm
- C6: renamed from C5; footprint (none) -> Capacitor_THT:C_Disc_D3.4mm_W2.1mm_P2.50mm
- C7: renamed from C3; footprint (none) -> Capacitor_THT:C_Disc_D3.4mm_W2.1mm_P2.50mm
- C8: renamed from C2; footprint (none) -> Capacitor_THT:C_Disc_D3.4mm_W2.1mm_P2.50mm
- D3: renamed from D1; footprint (none) -> LED_THT:LED_D1.8mm_W3.3mm_H2.4mm
- D4: renamed from D2; footprint (none) -> LED_THT:LED_D1.8mm_W3.3mm_H2.4mm
- D5: renamed from D4; footprint (none) -> LED_THT:LED_D1.8mm_W3.3mm_H2.4mm
- J1: renamed from J3; footprint (none) -> Connector_USB:USB_Micro-B_Molex_47346-0001
- J3: renamed from J1; value Conn_01x13_Pin -> LADO A; footprint Connector_PinHeader_2.54mm:PinHeader_1x13_P2.54mm_Vertical -> Connector_PinHeader_2.54mm:PinHeader_1x15_P2.54mm_Vertical
- J4: value Conn_01x13_Pin -> LADO B; footprint Connector_PinHeader_2.54mm:PinHeader_1x13_P2.54mm_Vertical -> Connector_PinHeader_2.54mm:PinHeader_1x16_P2.54mm_Vertical
- JP1: footprint (none) -> TestPoint:TestPoint_2Pads_Pitch2.54mm_Drill0.8mm
- R1: renamed from R10; footprint (none) -> Resistor_THT:R_Axial_DIN0204_L3.6mm_D1.6mm_P5.08mm_Horizontal
- R10: renamed from R1; footprint (none) -> Resistor_THT:R_Axial_DIN0204_L3.6mm_D1.6mm_P5.08mm_Horizontal
- R11: renamed from R4; footprint (none) -> Resistor_THT:R_Axial_DIN0204_L3.6mm_D1.6mm_P5.08mm_Horizontal
- R12: renamed from R5; footprint (none) -> Resistor_THT:R_Axial_DIN0204_L3.6mm_D1.6mm_P5.08mm_Horizontal
- R13: renamed from R3; footprint (none) -> Resistor_THT:R_Axial_DIN0204_L3.6mm_D1.6mm_P5.08mm_Horizontal
- R2, R6: footprint (none) -> Resistor_THT:R_Axial_DIN0204_L3.6mm_D1.6mm_P5.08mm_Horizontal
- R3: renamed from R12; footprint (none) -> Resistor_THT:R_Axial_DIN0204_L3.6mm_D1.6mm_P5.08mm_Horizontal
- R4: renamed from R7; footprint (none) -> Resistor_THT:R_Axial_DIN0204_L3.6mm_D1.6mm_P5.08mm_Horizontal
- R5: renamed from R9; footprint (none) -> Resistor_THT:R_Axial_DIN0204_L3.6mm_D1.6mm_P5.08mm_Horizontal
- R7: renamed from R8; footprint (none) -> Resistor_THT:R_Axial_DIN0204_L3.6mm_D1.6mm_P5.08mm_Horizontal
- R8: renamed from R13; footprint (none) -> Resistor_THT:R_Axial_DIN0204_L3.6mm_D1.6mm_P5.08mm_Horizontal
- R9: renamed from R11; footprint (none) -> Resistor_THT:R_Axial_DIN0204_L3.6mm_D1.6mm_P5.08mm_Horizontal
- SW1: renamed from SW2; footprint (none) -> Button_Switch_THT:SW_PUSH_6mm_H4.3mm
- SW2: renamed from SW3; footprint (none) -> Button_Switch_THT:SW_PUSH_6mm
- SW3: renamed from SW1; footprint (none) -> Button_Switch_THT:SW_PUSH_6mm
- U3: renamed from U1; footprint PDIP40_600MC_MCH -> PIC18L45K50:PDIP40_600MC_MCH
- renumbered D6 to D1, D5 to D2, D7 to D6, D8 to D7, D3 to D8, U3 to U1
